File: kicad/wii-daughterboard.sch (KiCad schematic (older format))
At the start: 40 parts, among them J1 Data, J10 A/V Pwr, J11 BT Sync, J12 Fan Pwr, J2 DC In, J3 WaveBird 1, J4 WaveBird 2, J5 Bluetooth, J6 GC 3/4, J7 Mobo Pwr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

Commit message: v3.0
Parts:
- removed J8: USB, Connector_JST:JST_SH_BM04B-SRSS-TB_1x04-1MP_P1.00mm_Vertical, symbol Connector_Generic_MountingPin:Conn_01x04_MountingPin
- removed TP1: 5V, TestPoint:TestPoint_Pad_D1.0mm, symbol Connector:TestPoint
- removed TP2: 3V3, TestPoint:TestPoint_Pad_D1.0mm, symbol Connector:TestPoint
- removed TP3: 1V15, TestPoint:TestPoint_Pad_D1.0mm, symbol Connector:TestPoint
- removed TP4: 1V0, TestPoint:TestPoint_Pad_D1.0mm, symbol Connector:TestPoint
- added C7, C8, C9: C, Capacitor_SMD:C_0603_1608Metric_Pad1.05x0.95mm_HandSolder, symbol Device:C
- added D1: D, Diode_SMD:D_SOD-123, symbol Device:D
- C1, C2, C3, C4, C5, C6: footprint Capacitor_SMD:C_0805_2012Metric_Pad1.15x1.40mm_HandSolder -> Capacitor_SMD:C_0603_1608Metric_Pad1.05x0.95mm_HandSolder
- J1: footprint Connector_JST:JST_SH_BM09B-SRSS-TB_1x09-1MP_P1.00mm_Vertical -> Connector_JST:JST_SH_BM07B-SRSS-TB_1x07-1MP_P1.00mm_Vertical; symbol Connector_Generic_MountingPin:Conn_01x09_MountingPin -> Connector_Generic:Conn_01x07
- J10: value A/V Pwr -> A/V; footprint Connector_JST:JST_PH_B2B-PH-SM4-TB_1x02-1MP_P2.00mm_Vertical -> Connector_JST:JST_SH_BM02B-SRSS-TB_1x02-1MP_P1.00mm_Vertical
- J11: value BT Sync -> Sync
- J12: value Fan Pwr -> Fan
- J2: value DC In -> DC
- J3: value WaveBird 1 -> GC 1; symbol Connector_Generic_MountingPin:Conn_01x03_MountingPin -> Connector_Generic:Conn_01x03
- J4: value WaveBird 2 -> GC 2; symbol Connector_Generic_MountingPin:Conn_01x03_MountingPin -> Connector_Generic:Conn_01x03
- J6: symbol Connector_Generic_MountingPin:Conn_01x05_MountingPin -> Connector_Generic:Conn_01x05
- J7: footprint Connector_JST:JST_PH_B4B-PH-SM4-TB_1x04-1MP_P2.00mm_Vertical -> Connector_JST:JST_PH_S4B-PH-SM4-TB_1x04-1MP_P2.00mm_Horizontal
- J9: symbol Connector_Generic_MountingPin:Conn_01x04_MountingPin -> Connector_Generic:Conn_01x04
- L1, L2, L3: footprint Inductor_SMD:L_Taiyo-Yuden_NR-40xx_HandSoldering -> project-footprints:INDPM3630X200N
- R9: footprint (none) -> Resistor_SMD:R_0603_1608Metric_Pad1.05x0.95mm_HandSolder
Connections:
- net USB_D+ is gone; now on net BT_D-: J1.1 (Pin_1)
- net USB_D- is gone; now on net BT_D+: J1.2 (Pin_2)
- net +1V0: now also J7.2 (Pin_2); no longer J7.3 (Pin_3)
- net +1V15: now also J7.3 (Pin_3); no longer J7.2 (Pin_2)
- net +3V3: now also J7.4 (Pin_4), C7.2, C8.2; no longer J7.1 (Pin_1)
- net +5V: now also D1.2 (A); no longer J10.1 (Pin_1)
- net BT_D+: no longer J1.8 (Pin_8)
- net BT_D-: no longer J1.9 (Pin_9)
- net GC_1: now also J1.4 (Pin_4); no longer J1.6 (Pin_6)
- net GC_3: now also J1.6 (Pin_6); no longer J1.4 (Pin_4)
- net GC_4: now also J1.7 (Pin_7); no longer J1.3 (Pin_3)
- net GND: now also J7.1 (Pin_1), C7.1, C8.1, C9.1; no longer J7.4 (Pin_4)
- net RST: now also J1.3 (Pin_3); no longer J1.7 (Pin_7)
- new net: C9.2, D1.1 (K), J10.1 (Pin_1)
- no-connect marks 12 -> 6
Other:
- note removed: "Test Points"
- note removed: "USB Header"
- moved on the sheet: H1, H2, J10, J11, J12, J7
